Commit message: Customize BCR Arm multitask MoveIt Gazebo simulation

File: bcr_arm_description/urdf/control/ros2_control.urdf.xacro (robot description, xacro)
@@ -5,8 +5,10 @@
       <hardware>
         <plugin>gz_ros2_control/GazeboSimSystem</plugin>
+        <param name="position_proportional_gain">200.0</param>
       </hardware>
+      <!-- ================= BCR Arm Joints ================= -->
       <joint name="joint1">
         <command_interface name="position"/>
-        <state_interface name="position" />
+        <state_interface name="position"/>
         <state_interface name="velocity"/>
         <state_interface name="effort"/>
@@ -48,4 +50,23 @@
         <state_interface name="effort"/>
       </joint>
+      <!-- ================= Simple Parallel Gripper Joints ================= -->
+      <joint name="simple_left_finger_joint">
+        <command_interface name="position">
+          <param name="min">0.0</param>
+          <param name="max">0.045</param>
+        </command_interface>
+        <state_interface name="position"/>
+        <state_interface name="velocity"/>
+        <state_interface name="effort"/>
+      </joint>
+      <joint name="simple_right_finger_joint">
+        <command_interface name="position">
+          <param name="min">0.0</param>
+          <param name="max">0.045</param>
+        </command_interface>
+        <state_interface name="position"/>
+        <state_interface name="velocity"/>
+        <state_interface name="effort"/>
+      </joint>
     </ros2_control>
   </xacro:macro>

File: bcr_arm_description/urdf/robots/bcr_arm.urdf.xacro (robot description, xacro)
@@ -1,10 +1,17 @@
 <?xml version="1.0"?>
 <robot xmlns:xacro="http://www.ros.org/wiki/xacro" name="bcr_arm">
-  <!-- Arguments -->
+  <!-- ================= Arguments ================= -->
   <xacro:arg name="use_gazebo" default="true"/>
   <xacro:arg name="ros2_controllers_path" default="bcr_arm_moveit_config/config/bcr_arm/ros2_controllers.yaml"/>
   <xacro:arg name="use_camera" default="true"/>
+  <xacro:arg name="use_gripper" default="true"/>
   <xacro:arg name="prefix" default=""/>
-  <!-- Material definitions for RViz -->
+  <!-- ================= Includes ================= -->
+  <xacro:include filename="$(find bcr_arm_description)/urdf/mech/bcr_arm_mech.urdf.xacro"/>
+  <xacro:include filename="$(find bcr_arm_description)/urdf/sensors/depth_camera.urdf.xacro"/>
+  <xacro:include filename="$(find bcr_arm_description)/urdf/control/gazebo_sim_ros2_control.urdf.xacro"/>
+  <xacro:include filename="$(find bcr_arm_description)/urdf/control/ros2_control.urdf.xacro"/>
+  <xacro:include filename="$(find bcr_arm_description)/urdf/end_effectors/simple_parallel_gripper.urdf.xacro"/>
+  <!-- ================= Materials ================= -->
   <material name="black">
     <color rgba="0.165 0.165 0.165 1.0"/>
@@ -16,5 +23,5 @@
     <color rgba="0.565 0.565 0.565 1.0"/>
   </material>
-  <!-- Connect to world frame -->
+  <!-- ================= World Frame ================= -->
   <link name="world"/>
   <joint name="world_to_base" type="fixed">
@@ -23,17 +30,24 @@
     <origin xyz="0 0 0" rpy="0 0 0"/>
   </joint>
-  <!-- Mechanical Arm -->
-  <xacro:include filename="$(find bcr_arm_description)/urdf/mech/bcr_arm_mech.urdf.xacro"/>
+  <!-- ================= Mechanical Arm ================= -->
   <xacro:bcr_arm_kinematics/>
-  <!-- Sensors -->
+  <!-- ================= Sensors ================= -->
   <xacro:if value="$(arg use_camera)">
-    <xacro:include filename="$(find bcr_arm_description)/urdf/sensors/depth_camera.urdf.xacro"/>
-    <xacro:depth_camera prefix="$(arg prefix)" parent_link="flange"/>
+    <xacro:depth_camera
+      prefix="$(arg prefix)"
+      parent_link="flange"/>
   </xacro:if>
-  <!-- ROS2 Control -->
+  <!-- ================= End Effector ================= -->
+  <xacro:simple_parallel_gripper
+    prefix="$(arg prefix)"
+    parent_link="flange"
+    xyz="0 0 0.055"
+    rpy="0 0 0"/>
+  <!-- ================= ROS2 Control ================= -->
   <xacro:if value="$(arg use_gazebo)">
-    <xacro:include filename="$(find bcr_arm_description)/urdf/control/gazebo_sim_ros2_control.urdf.xacro"/>
-    <xacro:load_gazebo_sim_ros2_control_plugin robot_name="bcr_arm" ros2_controllers_path="$(arg ros2_controllers_path)" use_gazebo="$(arg use_gazebo)"/>
-    <xacro:include filename="$(find bcr_arm_description)/urdf/control/ros2_control.urdf.xacro" />
+    <xacro:load_gazebo_sim_ros2_control_plugin
+      robot_name="bcr_arm"
+      ros2_controllers_path="$(arg ros2_controllers_path)"
+      use_gazebo="$(arg use_gazebo)"/>
     <xacro:ros2_control_interfaces/>
   </xacro:if>

File: bcr_arm_moveit_config/config/bcr_arm.ros2_control.xacro (robot description, xacro)
@@ -7,5 +7,5 @@
                 <xacro:if value="${ros2_control_hardware_type == 'mock_components'}">
                     <plugin>mock_components/GenericSystem</plugin>
-                </xacro:if>
+              </xacro:if>
                 <xacro:if value="${ros2_control_hardware_type == 'isaac'}">
                     <plugin>topic_based_ros2_control/TopicBasedSystem</plugin>
