Commit message: Add depth camera perception workflow

File: bcr_arm_description/urdf/robots/bcr_arm.urdf.xacro (robot description, xacro)
@@ -32,10 +32,4 @@
   <!-- ================= Mechanical Arm ================= -->
   <xacro:bcr_arm_kinematics/>
-  <!-- ================= Sensors ================= -->
-  <xacro:if value="$(arg use_camera)">
-    <xacro:depth_camera
-      prefix="$(arg prefix)"
-      parent_link="flange"/>
-  </xacro:if>
   <!-- ================= End Effector ================= -->
   <xacro:simple_parallel_gripper
@@ -44,4 +38,12 @@
     xyz="0 0 0.055"
     rpy="0 0 0"/>
+  <!-- ================= Sensors ================= -->
+  <xacro:if value="$(arg use_camera)">
+    <xacro:depth_camera
+      prefix="$(arg prefix)"
+      parent_link="world"
+      mount_xyz="0.45 0.00 1.95"
+      mount_rpy="0 1.6 0"/>
+  </xacro:if>
   <!-- ================= ROS2 Control ================= -->
   <xacro:if value="$(arg use_gazebo)">

File: bcr_arm_description/urdf/sensors/depth_camera.urdf.xacro (robot description, xacro)
@@ -1,10 +1,12 @@
 <?xml version="1.0"?>
 <robot xmlns:xacro="http://www.ros.org/wiki/xacro">
-  <xacro:macro name="depth_camera" params="prefix parent_link namespace:=bcr_arm">
+  <xacro:macro
+    name="depth_camera"
+    params="prefix parent_link mount_xyz:='0.04 0 0.096125' mount_rpy:='0 0 0' namespace:=bcr_arm">
     <!-- Camera Mount and Link -->
     <joint name="${prefix}camera_mount_joint" type="fixed">
       <parent link="${parent_link}"/>
       <child link="${prefix}camera_base_link"/>
-      <origin xyz="0.04 0 0.096125" rpy="0 0 0"/>
+      <origin xyz="${mount_xyz}" rpy="${mount_rpy}"/>
     </joint>
     <link name="${prefix}camera_base_link">
@@ -41,7 +43,7 @@
     </joint>
     <link name="${prefix}camera_depth_optical_frame"/>
-    <!-- Ignition Gazebo Camera Plugin -->
+    <!-- Ignition Gazebo RGB-D Camera Plugin -->
     <gazebo reference="${prefix}camera_link">
-      <sensor type="camera" name="depth_camera">
+      <sensor type="rgbd_camera" name="depth_camera">
         <always_on>true</always_on>
         <update_rate>20</update_rate>
